File: hardware/IFB-40004-R02 - I2C_Toggle_Switch.brd (EAGLE design)
At the start: 20 x 17 mm, 23 parts, among them J3 CUTTABLE_JUMPER, J4 CUT_JUMPER_2X, U2 ATTINY841-MMHR

Commit message: updated hardware files
Parts:
- removed J1, J2: (no value), SparkFun-Connectors:1X04_1MM_RA
- added J5, J6: QWIICSIDE, PlayingWithFusion_JST:SM04B-SRSS-TB
- moved J4 5.49 mm to (3.76, 8.23), turned to 180 degrees
- moved R5 0.30 mm to (2.84, 8.43)
Connections:
- net GND: now also J5.1, J6.1; no longer J1.1, J2.1
- net SCL: now also J5.4, J6.4; no longer J1.4, J2.4
- net SDA: now also J5.3, J6.3; no longer J1.3, J2.3
- net VCC: now also J5.2, J6.2; no longer J1.2, J2.2
Routing:
- net N$3: track 11.8 -> 3.53 mm
- net N$2: track 11.0 -> 2.72 mm
- net SDA: track 38.1 -> 34.0 mm, vias 5 -> 3
- net MISO: track 13.2 -> 15.8 mm
- net VCC: track 50.9 -> 53.2 mm, vias 2 -> 5
- net SCL: track 29.0 -> 29.6 mm, vias 3 -> 0
