File: hardware/IFB-40004-R02 - I2C_Toggle_Switch.sch (EAGLE design)
At the start: 23 parts, among them J3 CUTTABLE_JUMPER, J4 CUT_JUMPER_2X, U2 ATTINY841-MMHR

Commit message: updated hardware files
Parts:
- removed J1, J2: (no value), SparkFun-Connectors:QWIIC_CONNECTORJS-1MM
- added J5, J6: QWIICSIDE, PlayingWithFusion_JST:QWIICSIDE
Connections:
- net GND: now also J5.1, J6.1; no longer J1.GND, J2.GND
- net SCL: now also J5.4, J6.4; no longer J1.SCL, J2.SCL
- net SDA: now also J5.3, J6.3; no longer J1.SDA, J2.SDA
- net VCC: now also J5.2, J6.2; no longer J1.VCC, J2.VCC
Changed lines of the file:
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@@
 <part name="P+3" library="supply1" library_urn="urn:adsk.eagle:library:371" deviceset="VCC" device=""/>
 <part name="U2" library="ATTINY841-MMHR" deviceset="ATTINY841-MMHR" device=""/>
-<part name="J1" library="SparkFun-Connectors" library_urn="urn:adsk.eagle:library:513" deviceset="QWIIC_CONNECTOR" device="JS-1MM" package3d_urn="urn:adsk.eagle:package:38096/1"/>
 <part name="GND2" library="supply1" library_urn="urn:adsk.eagle:library:371" deviceset="GND" device=""/>
 <part name="P+1" library="supply1" library_urn="urn:adsk.eagle:library:371" deviceset="VCC" device=""/>
@@
 <part name="R4" library="rcl" library_urn="urn:adsk.eagle:library:334" deviceset="R-US_" device="R0603" package3d_urn="urn:adsk.eagle:package:23555/3" value="10k"/>
 <part name="R5" library="rcl" library_urn="urn:adsk.eagle:library:334" deviceset="R-US_" device="R0603" package3d_urn="urn:adsk.eagle:package:23555/3" value="10k"/>
-<part name="J2" library="SparkFun-Connectors" library_urn="urn:adsk.eagle:library:513" deviceset="QWIIC_CONNECTOR" device="JS-1MM" package3d_urn="urn:adsk.eagle:package:38096/1"/>
 <part name="GND3" library="supply1" library_urn="urn:adsk.eagle:library:371" deviceset="GND" device=""/>
 <part name="P+2" library="supply1" library_urn="urn:adsk.eagle:library:371" deviceset="VCC" device=""/>
@@
 <part name="U$3" library="PlayingWithFusion_Breakout-Lib" library_urn="urn:adsk.eagle:library:16658049" deviceset="FIDUCIAL" device="" package3d_urn="urn:adsk.eagle:package:16658275/1"/>
 <part name="J4" library="PlayingWithFusion_Breakout-Lib" library_urn="urn:adsk.eagle:library:16658049" deviceset="CUT_JUMPER_2X" device="" package3d_urn="urn:adsk.eagle:package:21537277/1"/>
+<part name="J5" library="PlayingWithFusion_JST" library_urn="urn:adsk.eagle:library:13097115" deviceset="QWIIC" device="SIDE" package3d_urn="urn:adsk.eagle:package:13097145/4"/>
+<part name="J6" library="PlayingWithFusion_JST" library_urn="urn:adsk.eagle:library:13097115" deviceset="QWIIC" device="SIDE" package3d_urn="urn:adsk.eagle:package:13097145/4"/>
 </parts>
 <sheets>
@@
 <attribute name="VALUE" x="96.52" y="105.22" size="2.0828" layer="96" ratio="10" rot="SR0"/>
 </instance>
-<instance part="J1" gate="J1" x="17.78" y="22.86" smashed="yes">
-<attribute name="VALUE" x="12.7" y="17.526" size="1.778" layer="96" font="vector" align="top-left"/>
-<attribute name="NAME" x="12.7" y="30.734" size="1.778" layer="95" font="vector"/>
-</instance>
 <instance part="GND2" gate="1" x="25.4" y="12.7" smashed="yes">
 <attribute name="VALUE" x="22.86" y="10.16" size="1.778" layer="96"/>
@@
 <attribute name="VALUE" x="69.342" y="62.23" size="1.778" layer="96" rot="R90"/>
 </instance>
-<instance part="J2" gate="J1" x="50.8" y="22.86" smashed="yes">
-<attribute name="VALUE" x="45.72" y="17.526" size="1.778" layer="96" font="vector" align="top-left"/>
-<attribute name="NAME" x="45.72" y="30.734" size="1.778" layer="95" font="vector"/>
-</instance>
-<instance part="GND3" gate="1" x="58.42" y="12.7" smashed="yes">
-<attribute name="VALUE" x="55.88" y="10.16" size="1.778" layer="96"/>
-</instance>
-<instance part="P+2" gate="VCC" x="73.66" y="38.1" smashed="yes">
-<attribute name="VALUE" x="71.12" y="35.56" size="1.778" layer="96" rot="R90"/>
+<instance part="GND3" gate="1" x="83.82" y="12.7" smashed="yes">
+<attribute name="VALUE" x="81.28" y="10.16" size="1.778" layer="96"/>
+</instance>
+<instance part="P+2" gate="VCC" x="99.06" y="38.1" smashed="yes">
+<attribute name="VALUE" x="96.52" y="35.56" size="1.778" layer="96" rot="R90"/>
 </instance>
 <instance part="GND4" gate="1" x="162.56" y="60.96" smashed="yes">
@@
 <attribute name="NAME" x="73.025" y="78.74" size="1.778" layer="95" font="vector"/>
 </instance>
+<instance part="J5" gate="J1" x="15.24" y="25.4" smashed="yes" rot="R180">
+<attribute name="NAME" x="19.304" y="17.4244" size="1.778" layer="95" font="vector" ratio="12" rot="R180"/>
+</instance>
+<instance part="J6" gate="J1" x="73.66" y="25.4" smashed="yes" rot="R180">
+<attribute name="NAME" x="77.724" y="17.4244" size="1.778" layer="95" font="vector" ratio="12" rot="R180"/>
+</instance>
 </instances>
 <busses>
@@
 </segment>
 <segment>
-<pinref part="J1" gate="J1" pin="GND"/>
 <pinref part="GND2" gate="1" pin="GND"/>
-<wire x1="25.4" y1="20.32" x2="25.4" y2="15.24" width="0.1524" layer="91"/>
-</segment>
-<segment>
-<pinref part="J2" gate="J1" pin="GND"/>
+<wire x1="25.4" y1="15.24" x2="25.4" y2="20.32" width="0.1524" layer="91"/>
+<pinref part="J5" gate="J1" pin="1"/>
+<wire x1="25.4" y1="20.32" x2="22.86" y2="20.32" width="0.1524" layer="91"/>
+</segment>
+<segment>
 <pinref part="GND3" gate="1" pin="GND"/>
-<wire x1="58.42" y1="20.32" x2="58.42" y2="15.24" width="0.1524" layer="91"/>
+<pinref part="J6" gate="J1" pin="1"/>
+<wire x1="81.28" y1="20.32" x2="83.82" y2="20.32" width="0.1524" layer="91"/>
+<wire x1="83.82" y1="20.32" x2="83.82" y2="15.24" width="0.1524" layer="91"/>
 </segment>
 <segment>
@@
 </segment>
 <segment>
-<pinref part="J1" gate="J1" pin="VCC"/>
-<wire x1="25.4" y1="22.86" x2="40.64" y2="22.86" width="0.1524" layer="91"/>
 <pinref part="P+1" gate="VCC" pin="VCC"/>
+<wire x1="22.86" y1="22.86" x2="40.64" y2="22.86" width="0.1524" layer="91"/>
 <wire x1="40.64" y1="22.86" x2="40.64" y2="35.56" width="0.1524" layer="91"/>
-</segment>
-<segment>
-<pinref part="J2" gate="J1" pin="VCC"/>
-<wire x1="58.42" y1="22.86" x2="73.66" y2="22.86" width="0.1524" layer="91"/>
+<pinref part="J5" gate="J1" pin="2"/>
+</segment>
+<segment>
 <pinref part="P+2" gate="VCC" pin="VCC"/>
-<wire x1="73.66" y1="22.86" x2="73.66" y2="35.56" width="0.1524" layer="91"/>
+<wire x1="81.28" y1="22.86" x2="99.06" y2="22.86" width="0.1524" layer="91"/>
+<wire x1="99.06" y1="22.86" x2="99.06" y2="35.56" width="0.1524" layer="91"/>
+<pinref part="J6" gate="J1" pin="2"/>
 </segment>
 <segment>
@@
 </segment>
 <segment>
-<pinref part="J1" gate="J1" pin="SDA"/>
-<wire x1="25.4" y1="25.4" x2="33.02" y2="25.4" width="0.1524" layer="91"/>
+<wire x1="22.86" y1="25.4" x2="33.02" y2="25.4" width="0.1524" layer="91"/>
 <wire x1="33.02" y1="25.4" x2="33.02" y2="33.02" width="0.1524" layer="91"/>
 <label x="33.02" y="33.02" size="1.778" layer="95" rot="R90" xref="yes"/>
-</segment>
-<segment>
-<pinref part="J2" gate="J1" pin="SDA"/>
-<wire x1="58.42" y1="25.4" x2="66.04" y2="25.4" width="0.1524" layer="91"/>
-<wire x1="66.04" y1="25.4" x2="66.04" y2="33.02" width="0.1524" layer="91"/>
-<label x="66.04" y="33.02" size="1.778" layer="95" rot="R90" xref="yes"/>
+<pinref part="J5" gate="J1" pin="3"/>
+</segment>
+<segment>
+<wire x1="81.28" y1="25.4" x2="91.44" y2="25.4" width="0.1524" layer="91"/>
+<wire x1="91.44" y1="25.4" x2="91.44" y2="33.02" width="0.1524" layer="91"/>
+<label x="91.44" y="33.02" size="1.778" layer="95" rot="R90" xref="yes"/>
+<pinref part="J6" gate="J1" pin="3"/>
 </segment>
 </net>
@@
 </segment>
 <segment>
-<pinref part="J1" gate="J1" pin="SCL"/>
-<wire x1="25.4" y1="27.94" x2="27.94" y2="27.94" width="0.1524" layer="91"/>
+<wire x1="22.86" y1="27.94" x2="27.94" y2="27.94" width="0.1524" layer="91"/>
 <wire x1="27.94" y1="27.94" x2="27.94" y2="33.02" width="0.1524" layer="91"/>
 <label x="27.94" y="33.02" size="1.778" layer="95" rot="R90" xref="yes"/>
-</segment>
-<segment>
-<pinref part="J2" gate="J1" pin="SCL"/>
-<wire x1="58.42" y1="27.94" x2="60.96" y2="27.94" width="0.1524" layer="91"/>
-<wire x1="60.96" y1="27.94" x2="60.96" y2="33.02" width="0.1524" layer="91"/>
-<label x="60.96" y="33.02" size="1.778" layer="95" rot="R90" xref="yes"/>
-</segment>
-<segment>
+<pinref part="J5" gate="J1" pin="4"/>
+</segment>
+<segment>
+<wire x1="81.28" y1="27.94" x2="86.36" y2="27.94" width="0.1524" layer="91"/>
+<wire x1="86.36" y1="27.94" x2="86.36" y2="33.02" width="0.1524" layer="91"/>
+<label x="86.36" y="33.02" size="1.778" layer="95" rot="R90" xref="yes"/>
+<pinref part="J6" gate="J1" pin="4"/>
+</segment>
+<segment>
